File: placa/pcb y esquematico/owen proyecto reloj.kicad_pcb (KiCad board)
At the start: 2 copper layers, 134.8 x 74.9 mm, 75 parts, among them J1 Screw_Terminal_01x02, SW1 SW_DPDT_x2, SW2 SW_MEC_5G, SW3 SW_MEC_5G, U1 74LS47, U10 74LS90, U11 74LS90, U12 74LS90, U14 4081, U2 74LS47, U3 74LS47, U4 74LS47, U5 74LS47, U6 74LS47, U7 74LS90, U8 74LS90, U9 74LS90

Commit message: Add files via upload
Parts:
- removed SW1: SW_DPDT_x2, EESTN5:SW_SPDT_TH_Vertical
- added U13: 74AUC2G32, Package_DIP:DIP-14_W10.16mm, F.Cu at (94.6, 111.7)
- added U15: 4081, Package_DIP:DIP-14_W10.16mm, F.Cu at (122.2, 115.4)
- added U16: 4081, Package_DIP:DIP-14_W10.16mm, F.Cu at (141.8, 115.3)
- added U17: 4081, Package_DIP:DIP-14_W10.16mm, F.Cu at (186.7, 110.6)
- added U18: 74AUC2G32, Package_DIP:DIP-14_W10.16mm, F.Cu at (145.9, 120.1)
- added U19: 4081, Package_DIP:DIP-14_W10.16mm, F.Cu at (209.5, 110.6)
- R10, R11, R12, R13, R14, R15, R16, R17, R18, R19, R20, R21, R22, R23, R24, R25, R26, R27, R28, R29, R30, R31, R32, R33, R34, R35, R36, R37, R38, R39, R40, R41, R42, R43, R44, R45, R46, R47, R48, R49, R50, R51: footprint Resistor_THT:R_Axial_DIN0207_L6.3mm_D2.5mm_P7.62mm_Horizontal -> Resistor_SMD:R_1206_3216Metric_Pad1.30x1.75mm_HandSolder
- moved D1 22.7 mm to (88.4, 97.1), turned to 0 degrees
- moved H3 16.9 mm to (216.3, 122.9)
- moved H4 16.9 mm to (87.8, 122.9)
- moved R36 5.72 mm to (112.1, 60.5)
- moved R43 5.65 mm to (89.6, 60.5)
- moved R29 5.51 mm to (134.1, 60.5)
- moved R15 5.48 mm to (178.8, 60.5)
- moved R50 5.48 mm to (201.1, 60.5)
- moved R22 5.48 mm to (156.4, 60.5)
- moved R37 5.41 mm to (114.7, 60.5)
- moved R44 5.35 mm to (92.2, 60.5)
- moved R30 5.24 mm to (136.6, 60.5)
- moved R16 5.21 mm to (181.3, 60.5)
- moved R23 5.21 mm to (159.0, 60.5)
- moved R51 5.21 mm to (203.7, 60.5)
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Connections:
- net Entrada1 renamed Out
- U10 pad 2: GND -> Q1
- U10 pad 3: GND -> Q7
- U14 pad 1: Es1 -> Q19
- U14 pad 2: Es2 -> Q18
- U14 pad 5: Es3 -> Q11
- U14 pad 6: Es4 -> Q10
- U2 pad 1: Es2 -> Q18
- U2 pad 2: Es1 -> Q19
- U3 pad 1: Es4 -> Q10
- U3 pad 2: Es3 -> Q11
- U7 pad 2: GND -> Q1
- U7 pad 3: GND -> Q7
- U8 pad 2: Es2 -> R2
- U8 pad 3: Es1 -> R2
- U8 pad 8: Es1 -> Q19
- U8 pad 9: Es2 -> Q18
- U9 pad 2: Es4 -> R1
- U9 pad 3: Es3 -> R1
- U9 pad 8: Es3 -> Q11
- U9 pad 9: Es4 -> Q10
Routing:
- net Q7: track 35.7 -> 225.2 mm, vias 0 -> 9
- net Q1: track 50.5 -> 221.8 mm, vias 0 -> 7
- net R1: track 0.00 -> 132.4 mm, vias 0 -> 4
- net Q10: track 0.00 -> 119.5 mm
- net Q11: track 0.00 -> 111.2 mm, vias 0 -> 2
- net Q18: track 0.00 -> 92.7 mm, vias 0 -> 2
- net Q19: track 0.00 -> 84.5 mm, vias 0 -> 4
- net R2: track 0.00 -> 63.2 mm, vias 0 -> 2
- net Net-(U18-Pad2): track 0.00 -> 60.8 mm
- net Es1: track 60.2 -> 0.00 mm
- net Es2: track 50.9 -> 0.00 mm
- net Net-(U13-Pad2): track 0.00 -> 43.5 mm
- net Net-(U17-Pad4): track 0.00 -> 40.2 mm
- net Es3: track 34.7 -> 0.00 mm
- net Es4: track 33.8 -> 0.00 mm
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Other:
- board size 134.8 x 74.9 mm -> 134.8 x 87.9 mm
