File: placa/pcb y esquematico/owen proyecto reloj.kicad_sch (KiCad schematic)
At the start: 75 parts, among them J1 Screw_Terminal_01x02, SW1 SW_DPDT_x2, SW2 SW_MEC_5G, SW3 SW_MEC_5G, U1 74LS47, U10 74LS90, U11 74LS90, U12 74LS90, U14 4081, U2 74LS47, U3 74LS47, U4 74LS47, U5 74LS47, U6 74LS47, U7 74LS90, U8 74LS90, U9 74LS90

Commit message: Add files via upload
Parts:
- removed SW1: SW_DPDT_x2, EESTN5:SW_SPDT_TH_Vertical, symbol Switch:SW_DPDT_x2
- added U13, U18: 74AUC2G32, Package_DIP:DIP-14_W10.16mm, symbol 74xGxx:74AUC2G32
- added U15, U16, U17, U19: 4081, Package_DIP:DIP-14_W10.16mm, symbol 4xxx:4081
- R10, R11, R12, R13, R14, R15, R16, R17, R18, R19, R20, R21, R22, R23, R24, R25, R26, R27, R28, R29, R30, R31, R32, R33, R34, R35, R36, R37, R38, R39, R40, R41, R42, R43, R44, R45, R46, R47, R48, R49, R50, R51: footprint Resistor_THT:R_Axial_DIN0207_L6.3mm_D2.5mm_P7.62mm_Horizontal -> Resistor_SMD:R_1206_3216Metric_Pad1.30x1.75mm_HandSolder
Connections:
- net cp2 is gone; now on net Out: U7.14 (CP0)
- net GND: no longer U10.2 (R0(1)), U10.3 (R0(2)), U7.2 (R0(1)), U7.3 (R0(2))
- net Q1: now also U10.2 (R0(1)), U7.2 (R0(1)), U15.5
- net Q7: now also U10.3 (R0(2)), U7.3 (R0(2)), U15.6
- net Entrada1 renamed Out
- net Es1 renamed Q19
- net Q19: now also U19.6; no longer U8.3 (R0(2))
- net Es2 renamed Q18
- net Q18: now also U19.5; no longer U8.2 (R0(1))
- net Es3 renamed Q11
- net Q11: now also U16.6; no longer U9.3 (R0(2))
- net Es4 renamed Q10
- net Q10: now also U16.5; no longer U9.2 (R0(1))
- new net: U17.4, U18.1
- new net: U18.2, U19.4
- new net: U13.1, U15.4
- new net: U13.2, U16.4
- new net R1: U13.7, U17.5, U17.6, U9.2 (R0(1)), U9.3 (R0(2))
- new net R2: U18.7, U8.2 (R0(1)), U8.3 (R0(2))
Other:
- note added: "Sistema de reseteo"
- note removed: "Switch"
- moved on the sheet: AFF10, AFF11, AFF6, AFF7, AFF8, AFF9, C1, D1, H1, H2, H3, H4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
